File: ELECTRONICAL_MAIN_BOARD_32/PIC32.sch (KiCad schematic (older format))
At the start: 12 parts

Commit message: Routage 66%
Parts:
- removed U?: PIC32_64, symbol PIC32_64
- added R16, R17, R18, R19, R20, R21, R22, R23, R24, R25, R26, R27, R28, R29: 10K, symbol R
- added U1: PIC32MX795F512H, symbol PIC32MX795F512H
- C4: renamed from C21; value C -> 100n
- C5: renamed from C22; value C -> 100n
- C6: renamed from C23; value C -> 100n
- R3, R4, R6: renamed from R?; value R -> 1K
- R5: renamed from R?; value R -> 10K
- gave numbers to parts that had none: 1
- renumbered C17 to C1, C18 to C2, C19 to C3
Connections:
- net labels added: SW12, SW6
- net labels removed: SW14, SW15
- wire segments 74 -> 106
Other:
- note added: "INTERNAL\n"

Commit message: SCHEMA 100% PCB 100%
Parts:
- added C10, C11, C7, C8: 100n, symbol C
Connections:
- net +3.3V: now also C7.1, C8.1
- net +5V: now also C10.1, C11.1
- net GND: now also C10.2, C11.2, C7.2, C8.2
Other:
- moved on the sheet: C1, C2, C3, C4, C5, C6
