File: ELECTRONICAL_MAIN_BOARD_32/V1-30/PIC32.sch (KiCad schematic (older format))
At the start: 42 parts, among them U1 PIC32MX795F512H

Commit message: ELECTRONICAL MAIN BOARD V1-30 Ready for production
Parts:
- added U7: 24C512, ~, symbol 24C512
Connections:
- net labels added: SCL1-5V, SDA1-5V
- wire segments 131 -> 139
Other:
- note added: "DECOUPLING \nCAPACITY"
- note added: "EEPROM"
- note added: "I2C ADDRESS = 0x00"
- note removed: "FILTER CAPACITER"
