File: ELECTRONICAL_MAIN_BOARD_32/V1-30/ELECTRONICAL_MAIN_BOARD_32.kicad_pcb (KiCad board)
At the start: 2 copper layers, 233.9 x 101 mm, 232 parts, among them J1 SIL1, J2 SIL1, J3 SIL1, J4 SIL1, J5 RJ12, J6 SIL1, J7 SIL1, K1 CONN_3, K2 CONN_3, K3 CONN_3, K4 CONN_3, K5 CONN_3, K6 CONN_3, K7 CONN_3, P1 HE10-16, P10 CONN_2, P11 CONN_2, P14 CAVALIER, P15 CAVALIER, P2 CONN_4, P3 CONN_4, P4 CONN_4, P5 CONN_4, P6 CONN_4, P7 CONN_4, P8 CONN_2, P9 CONN_5, Q1 BSS123, Q2 BSS123, Q3 BSS123, Q4 BSS123, SW1 SWITCH_X_8, SW2 SW_PUSH_SMALL, SW3 SWITCH_X_8, U1 PIC32MX795F512H, U2 74LVCC3245, U3 74LVCC3245, U4 PCA9306, U5 PCA9306, U6 74LVCC3245, U7 24C512, U8 LM75A, U9 PCF8563, X1 CRYSTAL1

Commit message: mechanical motor board v0.1+ mechanical main board v1.0
Parts:
- removed the C1 at (253.0, 142.0)
- removed the C10 at (195.3, 101.0)
- removed the C11 at (231.0, 129.7)
- removed the C12 at (269.2, 141.1)
- removed the C13 at (263.3, 130.2)
- removed the C2 at (253.4, 129.6)
- removed the C3 at (230.6, 122.6)
- removed the C4 at (250.1, 142.0)
- removed the C5 at (216.6, 133.0)
- removed the C6 at (250.2, 128.1)
- removed the C7 at (212.3, 120.4)
- removed the C8 at (204.9, 112.6)
- removed the C9 at (243.7, 130.2)
- removed the D1 at (242.5, 61.8)
- removed the D10 at (191.9, 89.7)
- removed the D11 at (234.2, 61.7)
- removed the D12 at (268.1, 125.1)
- removed the D13 at (267.1, 149.4)
- removed the D2 at (245.3, 61.8)
- removed the D3 at (236.7, 61.7)
- removed the D4 at (239.6, 61.7)
- removed the D5 at (260.4, 102.6)
- removed the D7 at (191.9, 66.8)
- removed the D8 at (191.9, 74.5)
- removed the D9 at (191.9, 82.1)
- removed the J1 at (213.4, 54.8)
- removed the J2 at (213.5, 149.0)
- removed the J3 at (259.3, 149.1)
- removed the J4 at (185.7, 54.8)
- removed the J5 at (255.2, 115.4)
- removed the J6 at (252.8, 54.5)
- removed the J7 at (185.7, 143.0)
- removed the K1 at (186.3, 66.2)
- removed the K2 at (186.3, 74.3)
- removed the K3 at (186.3, 82.4)
- removed the K4 at (186.3, 90.6)
- removed the K5 at (186.3, 114.9)
- removed the K6 at (186.3, 106.8)
- removed the K7 at (186.3, 98.7)
- removed the L1 at (197.5, 94.9)
- removed the P1 at (223.4, 139.6)
- removed the P10 at (214.9, 64.7)
- removed the P11 at (220.0, 64.7)
- removed the P14 at (237.0, 149.4)
- removed the P15 at (237.0, 145.8)
- removed the P2 at (198.0, 136.8)
- removed the P3 at (198.0, 126.1)
- removed the P4 at (186.3, 126.1)
- removed the P5 at (186.3, 136.8)
- removed the P6 at (244.3, 146.1)
- removed the P7 at (244.3, 132.6)
- removed the P8 at (266.9, 103.9)
- removed the P9 at (203.4, 65.8)
- removed the Q1 at (230.4, 97.7)
- removed the Q2 at (205.0, 101.1)
- removed the Q3 at (235.3, 127.3)
- removed the Q4 at (234.3, 100.2)
- removed the R1 at (236.7, 64.8)
- removed the R10 at (239.4, 128.4)
- removed the R11 at (256.9, 134.7)
- removed the R12 at (256.9, 136.5)
- removed the R13 at (241.3, 149.4)
- removed the R14 at (241.1, 146.4)
- removed the R16 at (263.6, 85.1)
- removed the R17 at (263.6, 82.5)
- removed the R18 at (263.6, 80.0)
- removed the R19 at (263.6, 77.4)
- removed the R2 at (239.6, 64.8)
- removed the R20 at (263.6, 71.8)
- removed the R21 at (263.6, 69.3)
- removed the R22 at (263.6, 66.8)
- removed the R23 at (263.6, 64.2)
- removed the R24 at (263.6, 61.7)
- removed the R25 at (263.6, 59.1)
- removed the R26 at (263.6, 95.2)
- removed the R27 at (263.6, 92.7)
- removed the R28 at (263.6, 90.1)
- removed the R29 at (263.6, 87.6)
- removed the R3 at (245.3, 64.7)
- removed the R30 at (194.8, 66.9)
- removed the R31 at (194.8, 74.5)
- removed the R32 at (194.8, 82.1)
- removed the R33 at (194.8, 89.8)
- removed the R34 at (197.5, 66.2)
- removed the R35 at (197.5, 73.8)
- removed the R36 at (197.5, 81.4)
- removed the R37 at (197.5, 89.0)
- removed the R38 at (243.9, 126.0)
- removed the R39 at (245.4, 141.1)
- removed the R4 at (242.5, 64.7)
- removed the R40 at (227.5, 98.9)
- removed the R41 at (203.2, 104.0)
- removed the R42 at (232.4, 126.5)
- removed the R43 at (229.7, 98.9)
- removed the R44 at (234.2, 64.8)
- removed the R45 at (266.1, 125.1)
- removed the R46 at (265.6, 144.5)
- removed the R5 at (260.9, 100.4)
- removed the R6 at (258.5, 102.6)
- removed the R7 at (258.5, 124.4)
- removed the R8 at (258.5, 126.3)
- removed the R9 at (241.4, 128.4)
- removed the RVAR1 at (204.3, 139.7)
- removed the SW1 at (264.8, 63.0)
- removed the SW2 at (266.0, 135.3)
- removed the SW3 at (264.8, 86.3)
- removed the U1 at (209.3, 100.3)
- removed the U2 at (212.0, 125.8)
- removed the U3 at (197.9, 108.1)
- removed the U4 at (249.5, 125.3)
- removed the U5 at (250.0, 139.3)
- removed the U6 at (225.0, 124.9)
- removed the U7 at (264.8, 141.2)
- removed the U8 at (224.5, 148.8)
- removed the U9 at (264.9, 140.5)
- removed the X1 at (256.4, 137.0)
Routing:
- net GND: track 1762.8 -> 881.4 mm, vias 56 -> 28
- net +5V: track 992.7 -> 496.4 mm, vias 42 -> 21
- net +3.3V: track 739.3 -> 369.6 mm, vias 24 -> 12
- net /5vto3v3/OC1-5V: track 298.0 -> 149.0 mm, vias 10 -> 5
- net /5vto3v3/SCL4: track 295.0 -> 147.5 mm, vias 12 -> 6
- net /PIC32/RST: track 278.2 -> 139.1 mm, vias 8 -> 4
- net +12V: track 246.9 -> 123.4 mm, vias 4 -> 2
- net /5vto3v3/RW: track 244.0 -> 122.0 mm, vias 6 -> 3
- net /5vto3v3/SDA4: track 208.2 -> 104.1 mm, vias 8 -> 4
- net /PIC32/PGED1: track 185.7 -> 92.8 mm, vias 4 -> 2
- net N-00000112: track 179.8 -> 89.9 mm, vias 4 -> 2
- net /5vto3v3/SDA1-5V: track 173.5 -> 86.7 mm, vias 6 -> 3
- net /5vto3v3/SCL1-5V: track 149.8 -> 74.9 mm, vias 8 -> 4
- net /5vto3v3/OC2-5V: track 147.6 -> 73.8 mm, vias 8 -> 4
- net /PIC32/SW5: track 145.8 -> 72.9 mm, vias 4 -> 2
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Other:
- board size 233.9 x 101 mm -> 88.5 x 100.3 mm
