File: MECHANICAL_MOTOR_BOARD/V1-00/Mechanical_Coder.sch (KiCad schematic (older format))
At the start: 29 parts, among them U2001 HCTL-2032, U2002 M74VHC1GT02DTT1G, X2001 12Mhz

Commit message: test mechanicalmotorboard PCB NOK
Parts:
- added Q2001: 2N7002, Housings_SOT-23_SOT-143_TSOT-6:SOT-23, symbol 2N7002
- added R2019: 1k, Resistors_SMD:R_0603, symbol R
- D2001, D2002, D2003, D2004, D2005, D2006: symbol LED -> LED-RESCUE-Mechanical_Motor_Board
- R2001, R2002, R2003, R2004, R2005, R2006, R2007, R2008, R2009, R2010, R2011, R2012: value 1.5k -> 2.1k; symbol R -> R-RESCUE-Mechanical_Motor_Board
- R2013: symbol R -> R-RESCUE-Mechanical_Motor_Board
- R2014, R2015, R2016, R2017, R2018: footprint (none) -> Resistors_SMD:R_0603; symbol R -> R-RESCUE-Mechanical_Motor_Board
- X2001: footprint Crystals_Oscillators_SMD:Resonator_7.2x3mm -> f4deb-mod-library:MDX75104
Connections:
- wire segments 87 -> 91
