File: BEACON_MAIN_BOARD/V0-10/BEACON_MAIN_BOARD V0-10.kicad_pcb (KiCad board)
At the start: 2 copper layers, 184 parts, among them J1 RJ12, K50 USBAB, P1 CONN_4, P2 CONN_4, P3 CONN_4, P4 CONN_4, P5 CONN_4, Q1 BSH202, Q2 2N7002, SW1 SW_PUSH_SMALL, SW2 SWITCH_INV, U1 PIC24FJ256GB206, U2 LM1117

Commit message: Beacon_Main_Board 50%
Parts:
- removed C1 (x2), C10 (x2), C2 (x2), C3 (x2), C4 (x2), C6 (x2), C9 (x2): 100n, SM0603_Capa
- removed C5 (x2), C7 (x2), C8 (x2): 10U/10V, SM1206
- removed COLONETTE (x8): VAL**, COLONETTE
- removed D1 (x2), D2 (x2): VERT, LED-0603
- removed D3 (x2): B340A, SM1206
- removed D4 (x2): JAUNE, LED-0603
- removed F1 (x2): FUSE, SM1206
- removed J1 (x2): RJ12, RJ12_CMS
- removed K50 (x2): USBAB, MICRO_USB_AB
- removed L1 (x2): 30Ohms, SM0603
- removed P1 (x2), P2 (x2), P3 (x2), P4 (x2), P5 (x2): CONN_4, KK-4
- removed PIN1 (x2), PIN10 (x2), PIN11 (x2), PIN12 (x2), PIN13 (x2), PIN14 (x2), PIN15 (x2), PIN16 (x2), PIN17 (x2), PIN18 (x2), PIN19 (x2), PIN2 (x2), PIN20 (x2), PIN21 (x2), PIN22 (x2), PIN23 (x2), PIN24 (x2), PIN25 (x2), PIN26 (x2), PIN27 (x2), PIN28 (x2), PIN29 (x2), PIN3 (x2), PIN30 (x2), PIN31 (x2), PIN32 (x2), PIN33 (x2), PIN34 (x2), PIN35 (x2), PIN36 (x2), PIN37 (x2), PIN38 (x2), PIN39 (x2), PIN4 (x2), PIN40 (x2), PIN41 (x2), PIN42 (x2), PIN43 (x2), PIN44 (x2), PIN45 (x2), PIN46 (x2), PIN5 (x2), PIN6 (x2), PIN7 (x2), PIN8 (x2), PIN9 (x2): CONN_1, 1pad
- removed Q1 (x2): BSH202, SOT23GDS
- removed Q2 (x2): 2N7002, SOT23GDS
- removed R1 (x2), R10 (x2), R11 (x2), R12 (x2), R7 (x2), R8 (x2), R9 (x2): 10k, SM0603_Resistor
- removed R2 (x2): 470, SM0603_Resistor
- removed R3 (x2): 3k3, SM0603_Resistor
- removed R4 (x2): 1k, SM0603_Resistor
- removed R5 (x2): 750, SM0603_Resistor
- removed R6 (x2): 100k, SM0603_Resistor
- removed RVAR1 (x2): 5k, POT_CMS
- removed SW1 (x2): SW_PUSH_SMALL, SW2
- removed SW2 (x2): SWITCH_INV, KK-3
- removed U1 (x2): PIC24FJ256GB206, TQFP_64
- removed U2 (x2): LM1117, DPAK
- added C2001: 100n, Capacitors_SMD:C_0603, F.Cu at (183.6, 105.3)
- added C2002: 10U/10V, Capacitors_Tantalum_SMD:TantalC_SizeA_EIA-3216_HandSoldering, F.Cu at (116.2, 105.9)
- added C2003: 100n, CEN-PCB:SM0603_Capa, F.Cu at (164.6, 90.0)
- added C2004: 100n, CEN-PCB:SM0603_Capa, F.Cu at (170.2, 101.0)
- added C2005: 100n, CEN-PCB:SM0603_Capa, F.Cu at (167.4, 101.3)
- added C2006: 100n, CEN-PCB:SM0603_Capa, F.Cu at (164.6, 101.3)
- added C2007: 10U/10V, Capacitors_Tantalum_SMD:TantalC_SizeA_EIA-3216_HandSoldering, B.Cu at (110.9, 83.8)
- added C3001: 100n, CEN-PCB:SM1206, B.Cu at (100.3, 94.7)
- added C3002: 100n, CEN-PCB:SM0603_Capa, B.Cu at (109.0, 105.7)
- added C3003: 100n, CEN-PCB:SM0603_Capa, B.Cu at (101.6, 115.3)
- added C3004: 100n, CEN-PCB:SM0603_Capa, B.Cu at (91.9, 102.9)
- added C3005: 10u/10V, Capacitors_Tantalum_SMD:TantalC_SizeA_EIA-3216_HandSoldering, F.Cu at (88.9, 111.6)
- added C3006: 100n, CEN-PCB:SM0603_Capa, B.Cu at (89.3, 109.0)
- added C3007: 10u/10V, Capacitors_Tantalum_SMD:TantalC_SizeA_EIA-3216_HandSoldering, B.Cu at (111.5, 105.2)
- added C3008: 22p, CEN-PCB:SM0603_Capa, B.Cu at (104.1, 83.6)
- added C3009: 22p, CEN-PCB:SM0603_Capa, B.Cu at (100.6, 83.6)
- added D1001: BLEU, LEDs:LED-0603, B.Cu at (89.9, 115.6)
- added D1002: ROUGE, LEDs:LED-0603, B.Cu at (88.1, 115.6)
- added D1003: JAUNE, LEDs:LED-0603, B.Cu at (86.4, 115.6)
- added D1004: VERT, LEDs:LED-0603, B.Cu at (84.6, 115.6)
- added D1005: BLEU, LEDs:LED-0603, F.Cu at (156.2, 104.6)
- added D1006: ROUGE, LEDs:LED-0603, F.Cu at (136.1, 95.0)
- added D1007: JAUNE, LEDs:LED-0603, F.Cu at (133.1, 95.0)
- added D1008: VERT, LEDs:LED-0603, F.Cu at (156.2, 108.5)
- added D1009: VERT, LEDs:LED-0603, B.Cu at (102.4, 66.8)
- added D1010: VERT, LEDs:LED-0603, B.Cu at (108.5, 78.4)
- added D2001: B340A, Diodes_SMD:SMA_Standard, F.Cu at (117.6, 74.2)
- added D3001: JAUNE, LEDs:LED-0603, B.Cu at (90.2, 119.9)
- added D3002: JAUNE, LEDs:LED-0603, B.Cu at (98.6, 119.9)
- added D3003: JAUNE, LEDs:LED-0603, B.Cu at (109.0, 124.6)
- added D3004: JAUNE, LEDs:LED-0603, B.Cu at (113.7, 124.7)
- added F2001: FUSE, Resistors_SMD:R_2010, F.Cu at (117.3, 69.1)
- added J1001: RJ12, 4deb-mod-library:RJ12, F.Cu at (95.5, 70.9)
- added J1002: RJ12, 4deb-mod-library:RJ12, F.Cu at (128.7, 70.7)
- added J1003: RJ45, Connect:RJ45_8, F.Cu at (139.3, 109.2)
- added K1001: CONN_3, CEN-PCB:KK-3, F.Cu at (95.2, 125.2)
- added K1002: CONN_3, CEN-PCB:KK-3, F.Cu at (103.6, 125.2)
- added K1005: CONN_3, CEN-PCB:KK-3, F.Cu at (142.9, 83.6)
- added K1006: CONN_3, CEN-PCB:KK-3, F.Cu at (142.9, 92.8)
- added K1009: USBAB, w_conn_pc:conn_usb_B_mini_smd, F.Cu at (111.9, 60.8)
- added K1010: COLONETTE, CEN-PCB:COLONETTE, F.Cu at (81.8, 123.7)
- added K1011: COLONETTE, CEN-PCB:COLONETTE, F.Cu at (142.0, 123.7)
- added K1012: COLONETTE, CEN-PCB:COLONETTE, F.Cu at (81.8, 63.5)
- added K1013: COLONETTE, CEN-PCB:COLONETTE, F.Cu at (142.0, 63.5)
- added L2001: 30Ohms, Resistors_SMD:R_0603, F.Cu at (125.9, 81.0)
- added P1001: CONN_5, CEN-PCB:KK-5, F.Cu at (80.0, 111.8)
- added P1002: CONN_4, 4deb-mod-library:KK-4, F.Cu at (80.0, 78.7)
- added P1003: CONN_4, 4deb-mod-library:KK-4, F.Cu at (80.0, 89.7)
- added P1004: CONN_4, 4deb-mod-library:KK-4, F.Cu at (80.0, 100.6)
- added P1005: CONN_4, 4deb-mod-library:KK-4, F.Cu at (134.6, 125.2)
- added Q2001: BSH202, CEN-PCB:SOT23GDS, F.Cu at (123.2, 74.3)
- added Q2002: 2N7002, TO_SOT_Packages_SMD:SOT-23, F.Cu at (123.1, 78.7)
- added Q3001: 2N7002, TO_SOT_Packages_SMD:SOT-23, B.Cu at (88.9, 74.7)
- added Q3002: 2N7002, TO_SOT_Packages_SMD:SOT-23, B.Cu at (88.9, 85.6)
- added Q3003: 2N7002, TO_SOT_Packages_SMD:SOT-23, B.Cu at (88.9, 96.4)
- added Q3004: 2N7002, TO_SOT_Packages_SMD:SOT-23, B.Cu at (88.9, 79.0)
- added Q3005: 2N7002, TO_SOT_Packages_SMD:SOT-23, B.Cu at (88.9, 89.9)
- added Q3006: 2N7002, TO_SOT_Packages_SMD:SOT-23, B.Cu at (88.9, 100.8)
- added Q3007: 2N7002, TO_SOT_Packages_SMD:SOT-23, B.Cu at (116.1, 99.3)
- added Q3008: 2N7002, TO_SOT_Packages_SMD:SOT-23, B.Cu at (116.1, 106.2)
- added Q3009: 2N7002, TO_SOT_Packages_SMD:SOT-23, B.Cu at (116.1, 102.7)
- added Q3010: 2N7002, TO_SOT_Packages_SMD:SOT-23, B.Cu at (116.1, 109.6)
- added R1001: 680, Resistors_SMD:R_0603, F.Cu at (171.3, 83.3)
- added R2002: 22k, Resistors_SMD:R_0603, B.Cu at (106.7, 118.0)
- added R2003: 10k, Resistors_SMD:R_0603, F.Cu at (131.6, 75.7)
- added R2004: 470, Resistors_SMD:R_0603, F.Cu at (163.5, 71.8)
- added R2005: 12k, Resistors_SMD:R_0603, B.Cu at (109.7, 118.0)
- added R2006: 1.5k, Resistors_SMD:R_0603, F.Cu at (168.8, 71.8)
- added R2007: 1.5k, Resistors_SMD:R_0603, F.Cu at (132.3, 98.3)
- added R2008: 1.5k, Resistors_SMD:R_0603, F.Cu at (182.4, 96.8)
- added R2009: 1.5k, Resistors_SMD:R_0603, F.Cu at (155.4, 111.4)
- added R2010: 12k, Resistors_SMD:R_0603, B.Cu at (130.8, 121.5)
- added R2011: 1.5k, Resistors_SMD:R_0603, F.Cu at (108.5, 82.7)
- added R2012: 22k, Resistors_SMD:R_0603, B.Cu at (127.8, 118.7)
- added R2013: 4.7k, Resistors_SMD:R_0603, B.Cu at (134.0, 118.7)
- added R2014: 100k, Resistors_SMD:R_0603, F.Cu at (123.1, 81.5)
- added R2015: 8.2k, Resistors_SMD:R_0603, F.Cu at (117.6, 77.7)
- added R2016: 2.2k, Resistors_SMD:R_0603, F.Cu at (119.5, 77.7)
- added R3001: 10k, Resistors_SMD:R_0603, B.Cu at (84.5, 74.5)
- added R3002: 10k, Resistors_SMD:R_0603, B.Cu at (84.5, 85.3)
- added R3003: 10k, Resistors_SMD:R_0603, B.Cu at (84.5, 96.3)
- added R3004: 10k, Resistors_SMD:R_0603, B.Cu at (91.8, 76.5)
- added R3005: 10k, Resistors_SMD:R_0603, B.Cu at (91.9, 85.7)
- added R3006: 10k, Resistors_SMD:R_0603, B.Cu at (91.9, 94.6)
- added R3007: 10k, Resistors_SMD:R_0603, F.Cu at (101.9, 43.5)
- added R3008: 0, Resistors_SMD:R_0603, B.Cu at (101.2, 79.1)
- added R3009: 12k, Resistors_SMD:R_0603, B.Cu at (84.8, 78.7)
- added R3010: 12k, Resistors_SMD:R_0603, B.Cu at (84.8, 89.7)
- added R3011: 12k, Resistors_SMD:R_0603, B.Cu at (84.8, 100.6)
- added R3012: 22k, Resistors_SMD:R_0603, B.Cu at (84.8, 80.5)
- added R3013: 22k, Resistors_SMD:R_0603, B.Cu at (84.8, 91.4)
- added R3014: 22k, Resistors_SMD:R_0603, B.Cu at (84.8, 102.4)
- added R3015: 470, Resistors_SMD:R_0603, B.Cu at (101.6, 70.1)
- added R3016: 680, Resistors_SMD:R_0603, B.Cu at (89.9, 112.5)
- added R3017: 680, Resistors_SMD:R_0603, B.Cu at (88.1, 112.5)
- added R3018: 680, Resistors_SMD:R_0603, B.Cu at (86.4, 112.5)
- added R3019: 680, Resistors_SMD:R_0603, B.Cu at (84.6, 112.5)
- added R3020: 10k, Resistors_SMD:R_0603, B.Cu at (120.1, 100.3)
- added R3021: 10k, Resistors_SMD:R_0603, B.Cu at (120.1, 107.2)
- added R3022: 10k, Resistors_SMD:R_0603, B.Cu at (120.1, 103.8)
- added R3023: 10k, Resistors_SMD:R_0603, B.Cu at (120.1, 110.6)
- added R3024: 1.5k, Resistors_SMD:R_0603, B.Cu at (92.2, 119.9)
- added R3025: 1.5k, Resistors_SMD:R_0603, B.Cu at (94.2, 119.9)
- added R3026: 1.5k, Resistors_SMD:R_0603, B.Cu at (100.6, 119.9)
- added R3027: 1.5k, Resistors_SMD:R_0603, B.Cu at (102.6, 119.9)
- added R3028: 1.5k, Resistors_SMD:R_0603, B.Cu at (109.0, 122.6)
- added R3029: 1.5k, Resistors_SMD:R_0603, B.Cu at (109.0, 120.5)
- added R3030: 1.5k, Resistors_SMD:R_0603, B.Cu at (113.7, 122.7)
- added R3031: 1.5k, Resistors_SMD:R_0603, B.Cu at (113.7, 120.7)
- added SW2001: SW_PUSH_SMALL, CEN-PCB:SW, F.Cu at (142.5, 70.4)
- added SW2002: SWITCH_INV, CEN-PCB:CAVALIER, F.Cu at (107.1, 69.7)
- added U2001: PIC24FJ256GB206, Housings_QFP:TQFP-64_10x10mm_Pitch0.5mm, F.Cu at (121.5, 91.6)
- added U3001: PIC32MX795F512H, Housings_QFP:TQFP-64_10x10mm_Pitch0.5mm, B.Cu at (101.0, 103.5)
- added X3001: 8Mhz, CEN-PCB:QTZ, B.Cu at (102.4, 88.6)
Routing:
- net +3.3V: track 528.5 -> 0.00 mm, vias 20 -> 0
- net GND: track 741.9 -> 334.0 mm, vias 24 -> 12
- net +5VD: track 466.2 -> 96.7 mm, vias 10 -> 7
- net +3V3: track 0.00 -> 91.5 mm, vias 0 -> 3
- net /USBID: track 91.1 -> 0.00 mm, vias 4 -> 0
- net /D+: track 80.4 -> 0.00 mm
- net /RX1: track 79.8 -> 0.00 mm
- net /VBUS: track 77.6 -> 0.00 mm, vias 2 -> 0
- net /D-: track 77.4 -> 0.00 mm
- net Net-(R3011-Pad1): track 0.00 -> 76.5 mm, vias 0 -> 2
- net N-0000040: track 75.3 -> 0.00 mm
- net /PGD: track 75.2 -> 0.00 mm, vias 2 -> 0
- net /TX1: track 69.1 -> 0.00 mm
- net /PGC: track 67.6 -> 0.00 mm, vias 2 -> 0
- net N-0000033: track 67.6 -> 0.00 mm
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- removed copper zone on B.Cu, net +3.3V
- removed copper zone on F.Cu, net +3.3V
- removed copper zone on B.Cu, net GND
- removed copper zone on F.Cu, net GND
Other:
- board outline added: 70.4 x 70.4 mm
- net class Default: trace_width 0.254 -> 0.25; via_dia 0.889 -> 0.6; via_drill 0.635 -> 0.4
- rule trace_min: 0.254 -> 0.2
- rule via_min_drill: 0.6 -> 0.3
- rule via_min_size: 0.889 -> 0.4
- board text added: "POWER"
- board text removed: "I2C POWER"
- board text removed: "IOIO_BOARD"
- board text removed: "ISP"
- board text removed: "P1"
- board text removed: "P10"
- board text removed: "P11"
- board text removed: "P12"
- board text removed: "P13"
- board text removed: "P14"
- board text removed: "P15"
- board text removed: "P16"
- board text removed: "P17"
- board text removed: "P18"
- board text removed: "P19"
- board text removed: "P2"
- board text removed: "P20"
- board text removed: "P21"
- board text removed: "P22"
- board text removed: "P23"
- board text removed: "P24"
- board text removed: "P25"
- board text removed: "P26"
- board text removed: "P27"
- board text removed: "P28"
- board text removed: "P29"
- board text removed: "P30"
- board text removed: "P31"
- board text removed: "P32"
- board text removed: "P33"
- board text removed: "P34"
- board text removed: "P37"
- board text removed: "P38"
- board text removed: "P39"
- board text removed: "P40"
- board text removed: "P41"
- board text removed: "P42"
- board text removed: "P43"
- board text removed: "P44"
- board text removed: "P45"
- board text removed: "P46"
- board text removed: "P8"
- board text removed: "P9"
- board text removed: "UART4"
- board text removed: "USB"
- board text removed: "V0-10 15/07"

Commit message: PCB 80%
Parts:
- C2007, C3007: footprint Capacitors_Tantalum_SMD:TantalC_SizeA_EIA-3216_HandSoldering -> Capacitors_Tantalum_SMD:TantalC_SizeA_EIA-3216_Wave
- D1005, D1006, D1007, D1008, R1001, R2003, R2006, R2007, R2008, R2009, R3007: moved to B.Cu
- moved C2001 71.0 mm to (116.3, 82.7), turned to 270 degrees
- moved R1001 67.5 mm to (105.9, 66.8)
- moved C2005 59.0 mm to (109.7, 88.9), turned to 90 degrees
- moved R2008 52.4 mm to (130.4, 90.0), turned to 90 degrees
- moved C2004 50.2 mm to (120.0, 101.0), turned to 180 degrees
- moved R2006 46.9 mm to (125.6, 90.0), turned to 90 degrees
- moved C2003 42.1 mm to (123.1, 83.2)
- moved D1005 35.3 mm to (125.6, 87.1), turned to 270 degrees
- moved C2006 34.6 mm to (131.7, 90.6), turned to 270 degrees
- moved R3008 31.9 mm to (89.5, 108.8)
- moved D1008 31.6 mm to (132.8, 87.1), turned to 270 degrees
- moved R2009 31.1 mm to (132.8, 90.0), turned to 90 degrees
- moved R2004 30.0 mm to (134.1, 77.9), turned to 270 degrees
- moved R3007 29.7 mm to (101.6, 73.3), turned to 270 degrees
- moved R2014 18.8 mm to (109.3, 94.4), turned to 270 degrees
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Connections:
- K1009 pad : (no net) -> GND
Routing:
- net GND: track 334.0 -> 488.7 mm, vias 12 -> 17
- net +BATT: track 0.00 -> 85.5 mm, vias 0 -> 2
- net +3V3: track 91.5 -> 176.4 mm, vias 3 -> 7
- net +5VD: track 96.7 -> 176.4 mm, vias 7 -> 10
- net Net-(Q3006-Pad1): track 2.10 -> 66.4 mm, vias 0 -> 2
- net +12V: track 64.9 -> 115.2 mm, vias 0 -> 2
- net /IOIO/HOST: track 6.54 -> 41.3 mm, vias 0 -> 2
- net /IOIO/PGC24: track 0.00 -> 22.8 mm, vias 0 -> 1
- net /IOIO/PGD24: track 0.00 -> 21.6 mm, vias 0 -> 1
- net Net-(R2004-Pad2): track 0.00 -> 20.2 mm
- net Net-(R2009-Pad1): track 4.40 -> 23.7 mm, vias 0 -> 1
- net Net-(R2008-Pad1): track 3.69 -> 20.7 mm, vias 0 -> 1
- net Net-(R2007-Pad1): track 2.73 -> 17.4 mm, vias 0 -> 1
- net +5V: track 0.00 -> 14.6 mm, vias 0 -> 3
- net Net-(R2006-Pad1): track 1.92 -> 14.5 mm, vias 0 -> 1
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
Commit message: ELECTRONICAL_MAIN_BOARD_32 V1-40
Parts:
- moved K1012 88.0 mm to (76.2, 151.3), turned to 90 degrees
- moved P1002 75.2 mm to (91.5, 153.1), turned to 180 degrees
- moved R3001 74.1 mm to (87.3, 148.6), turned to 0 degrees
- moved K1013 71.3 mm to (76.2, 91.1), turned to 90 degrees
- moved R3009 69.8 mm to (91.5, 148.2), turned to 270 degrees
- moved K1009 69.6 mm to (75.0, 121.2), turned to 270 degrees
- moved Q3001 69.5 mm to (87.4, 144.2), turned to 270 degrees
- moved R3012 68.2 mm to (93.2, 148.2), turned to 270 degrees
- moved D1009 67.9 mm to (79.5, 130.7), turned to 90 degrees
- moved J1001 67.8 mm to (83.6, 137.6), turned to 270 degrees
- moved P1003 67.2 mm to (102.4, 153.1), turned to 180 degrees
- moved R1001 65.9 mm to (79.5, 127.2), turned to 90 degrees
- moved Q3004 65.2 mm to (91.7, 144.2), turned to 270 degrees
- moved R3004 64.9 mm to (89.2, 141.3), turned to 180 degrees
- moved R3002 64.7 mm to (98.1, 148.6), turned to 0 degrees
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Routing:
- net +3V3: track 176.4 -> 363.9 mm, vias 7 -> 13
- net GND: track 488.7 -> 596.8 mm, vias 17 -> 26
- net +5VD: track 176.4 -> 258.2 mm, vias 10 -> 13
- net Net-(R3011-Pad1): track 78.5 -> 65.4 mm
- net Net-(Q3006-Pad1): track 66.4 -> 53.5 mm
- net Net-(R3015-Pad1): track 57.3 -> 64.4 mm
- net /IOIO/TX4: track 61.8 -> 58.0 mm
- net Net-(R3009-Pad1): track 34.6 -> 31.1 mm
- net +BATT: track 85.5 -> 88.9 mm
- net /IOIO/TX1: track 27.7 -> 25.2 mm
- net Net-(R3026-Pad2): track 16.7 -> 19.1 mm
- net /IOIO/RX424: track 75.0 -> 77.0 mm
- net Net-(R3010-Pad1): track 56.6 -> 54.8 mm
- net Net-(R3024-Pad2): track 14.2 -> 16.0 mm
- net /PIC32MX795F512H/LASER2: track 4.58 -> 2.81 mm
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- added copper zone on B.Cu, net GND
- added copper zone on F.Cu, net GND
Other:
- board text added: "3.3V"
- board text added: "BEACON_MAIN_BOARD V0-10 DEC 2015 F4DEB"
- board text added: "HOST"
- board text added: "LAS1"
- board text added: "LAS3"
- board text added: "LAS4"
- board text added: "PIC24"
- board text added: "PIC32"
- board text added: "PWM1"
- board text added: "PWM2"
- board text added: "STATUS"
- board text added: "UART IOIO"
- board text added: "UART4"
- board text removed: "UART1"
