File: ICD_BOARD/V0-10/ICD_BOARD.kicad_pcb (KiCad board)
At the start: 2 copper layers, 82.5 x 118.1 mm, 24 parts, among them J1001 RJ12, J1002 RJ12, J1003 RJ12, J1004 RJ12, J1005 RJ12, J1006 RJ12, J1007 RJ12, J1008 RJ12, K1001 COLONETTE, K1002 COLONETTE, K1003 COLONETTE, K1004 COLONETTE

Commit message: MAJ ICD BOARD + 3D Mechanical Power Board V0.10
Parts:
- removed the J1001 at (50.8, 147.3)
- removed the J1002 at (50.8, 152.4)
- removed the J1003 at (66.0, 147.3)
- removed the J1004 at (66.0, 152.4)
- removed the J1005 at (81.3, 147.3)
- removed the J1006 at (81.3, 152.4)
- removed the J1007 at (96.5, 147.3)
- removed the J1008 at (96.5, 152.4)
- removed the K1001 at (38.1, 158.8)
- removed the K1002 at (109.2, 141.0)
- removed the K1003 at (38.1, 141.0)
- removed the K1004 at (109.2, 158.8)
- moved J1001 1.65 mm to (52.1, 63.9)
Connections:
- J1001 pad 7: (no net) -> Net-(J1001-Pad7)
- J1001 pad 8: (no net) -> Net-(J1001-Pad8)
- J1002 pad 1: Net-(J1001-Pad6) -> Net-(J1001-Pad1)
- J1002 pad 2: Net-(J1001-Pad5) -> Net-(J1001-Pad2)
- J1002 pad 3: Net-(J1001-Pad4) -> Net-(J1001-Pad3)
- J1002 pad 4: Net-(J1001-Pad3) -> Net-(J1001-Pad4)
- J1002 pad 5: Net-(J1001-Pad2) -> Net-(J1001-Pad5)
- J1002 pad 6: Net-(J1001-Pad1) -> Net-(J1001-Pad6)
- J1002 pad 7: (no net) -> Net-(J1002-Pad7)
- J1002 pad 8: (no net) -> Net-(J1002-Pad8)
- J1003 pad 7: (no net) -> Net-(J1003-Pad7)
- J1003 pad 8: (no net) -> Net-(J1003-Pad8)
- J1004 pad 1: Net-(J1003-Pad6) -> Net-(J1003-Pad1)
- J1004 pad 2: Net-(J1003-Pad5) -> Net-(J1003-Pad2)
- J1004 pad 3: Net-(J1003-Pad4) -> Net-(J1003-Pad3)
- J1004 pad 4: Net-(J1003-Pad3) -> Net-(J1003-Pad4)
- J1004 pad 5: Net-(J1003-Pad2) -> Net-(J1003-Pad5)
- J1004 pad 6: Net-(J1003-Pad1) -> Net-(J1003-Pad6)
- J1004 pad 7: (no net) -> Net-(J1004-Pad7)
- J1004 pad 8: (no net) -> Net-(J1004-Pad8)
- J1005 pad 7: (no net) -> Net-(J1005-Pad7)
- J1005 pad 8: (no net) -> Net-(J1005-Pad8)
- J1006 pad 1: Net-(J1005-Pad6) -> Net-(J1005-Pad1)
- J1006 pad 2: Net-(J1005-Pad5) -> Net-(J1005-Pad2)
- J1006 pad 3: Net-(J1005-Pad4) -> Net-(J1005-Pad3)
- J1006 pad 4: Net-(J1005-Pad3) -> Net-(J1005-Pad4)
- J1006 pad 5: Net-(J1005-Pad2) -> Net-(J1005-Pad5)
- J1006 pad 6: Net-(J1005-Pad1) -> Net-(J1005-Pad6)
- J1006 pad 7: (no net) -> Net-(J1006-Pad7)
- J1006 pad 8: (no net) -> Net-(J1006-Pad8)
- J1007 pad 7: (no net) -> Net-(J1007-Pad7)
- J1007 pad 8: (no net) -> Net-(J1007-Pad8)
- J1008 pad 1: Net-(J1007-Pad6) -> Net-(J1007-Pad1)
- J1008 pad 2: Net-(J1007-Pad5) -> Net-(J1007-Pad2)
- J1008 pad 3: Net-(J1007-Pad4) -> Net-(J1007-Pad3)
- J1008 pad 4: Net-(J1007-Pad3) -> Net-(J1007-Pad4)
- J1008 pad 5: Net-(J1007-Pad2) -> Net-(J1007-Pad5)
- J1008 pad 6: Net-(J1007-Pad1) -> Net-(J1007-Pad6)
- J1008 pad 7: (no net) -> Net-(J1008-Pad7)
- J1008 pad 8: (no net) -> Net-(J1008-Pad8)
Routing:
- net Net-(J1007-Pad6): track 15.2 -> 0.00 mm
- net Net-(J1007-Pad5): track 15.2 -> 0.00 mm
- net Net-(J1007-Pad4): track 15.2 -> 0.00 mm
- net Net-(J1007-Pad3): track 15.2 -> 0.00 mm
- net Net-(J1007-Pad2): track 15.2 -> 0.00 mm
- net Net-(J1007-Pad1): track 15.2 -> 0.00 mm
- net Net-(J1005-Pad6): track 15.2 -> 0.00 mm
- net Net-(J1005-Pad5): track 15.2 -> 0.00 mm
- net Net-(J1005-Pad4): track 15.2 -> 0.00 mm
- net Net-(J1005-Pad3): track 15.2 -> 0.00 mm
- net Net-(J1005-Pad2): track 15.2 -> 0.00 mm
- net Net-(J1005-Pad1): track 15.2 -> 0.00 mm
- net Net-(J1003-Pad6): track 15.2 -> 0.00 mm
- net Net-(J1003-Pad5): track 15.2 -> 0.00 mm
- net Net-(J1003-Pad4): track 15.2 -> 0.00 mm
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- removed copper zone on B.Cu, net (none)
- removed copper zone on F.Cu, net (none)
Other:
- board size 82.5 x 118.1 mm -> 81.3 x 34.2 mm

Commit message: MAJ CONNECTORS_BOARD V0-20
Parts:
- moved J1001 164.8 mm to (214.6, 36.7)
- moved J1003 164.6 mm to (229.9, 36.7)
- moved J1005 164.6 mm to (245.1, 36.7)
- moved J1007 164.6 mm to (260.4, 36.7)
- moved K1001 164.6 mm to (201.9, 25.3)
- moved K1004 164.6 mm to (273.1, 25.3)
- moved J1002 164.2 mm to (214.6, 34.2)
- moved J1004 164.2 mm to (229.9, 34.2)
- moved J1006 164.2 mm to (245.1, 34.2)
- moved J1008 164.2 mm to (260.4, 34.2)
- moved K1002 164.2 mm to (273.1, 45.6)
- moved K1003 164.2 mm to (201.9, 45.6)
Connections:
- J1002 pad 1: Net-(J1001-Pad1) -> Net-(J1001-Pad6)
- J1002 pad 2: Net-(J1001-Pad2) -> Net-(J1001-Pad5)
- J1002 pad 3: Net-(J1001-Pad3) -> Net-(J1001-Pad4)
- J1002 pad 4: Net-(J1001-Pad4) -> Net-(J1001-Pad3)
- J1002 pad 5: Net-(J1001-Pad5) -> Net-(J1001-Pad2)
- J1002 pad 6: Net-(J1001-Pad6) -> Net-(J1001-Pad1)
- J1004 pad 1: Net-(J1003-Pad1) -> Net-(J1003-Pad6)
- J1004 pad 2: Net-(J1003-Pad2) -> Net-(J1003-Pad5)
- J1004 pad 3: Net-(J1003-Pad3) -> Net-(J1003-Pad4)
- J1004 pad 4: Net-(J1003-Pad4) -> Net-(J1003-Pad3)
- J1004 pad 5: Net-(J1003-Pad5) -> Net-(J1003-Pad2)
- J1004 pad 6: Net-(J1003-Pad6) -> Net-(J1003-Pad1)
- J1006 pad 1: Net-(J1005-Pad1) -> Net-(J1005-Pad6)
- J1006 pad 2: Net-(J1005-Pad2) -> Net-(J1005-Pad5)
- J1006 pad 3: Net-(J1005-Pad3) -> Net-(J1005-Pad4)
- J1006 pad 4: Net-(J1005-Pad4) -> Net-(J1005-Pad3)
- J1006 pad 5: Net-(J1005-Pad5) -> Net-(J1005-Pad2)
- J1006 pad 6: Net-(J1005-Pad6) -> Net-(J1005-Pad1)
- J1008 pad 1: Net-(J1007-Pad1) -> Net-(J1007-Pad6)
- J1008 pad 2: Net-(J1007-Pad2) -> Net-(J1007-Pad5)
- J1008 pad 3: Net-(J1007-Pad3) -> Net-(J1007-Pad4)
- J1008 pad 4: Net-(J1007-Pad4) -> Net-(J1007-Pad3)
- J1008 pad 5: Net-(J1007-Pad5) -> Net-(J1007-Pad2)
- J1008 pad 6: Net-(J1007-Pad6) -> Net-(J1007-Pad1)
Routing:
- net Net-(J1001-Pad2): track 28.4 -> 5.08 mm
- net Net-(J1001-Pad4): track 28.3 -> 5.08 mm, vias 2 -> 0
- net Net-(J1001-Pad6): track 23.0 -> 5.08 mm, vias 2 -> 0
- net Net-(J1001-Pad1): track 13.1 -> 5.08 mm, vias 2 -> 0
- net Net-(J1001-Pad5): track 10.7 -> 5.08 mm, vias 2 -> 0
- net Net-(J1007-Pad6): track 0.00 -> 5.08 mm
- net Net-(J1007-Pad4): track 0.00 -> 5.08 mm
- net Net-(J1007-Pad2): track 0.00 -> 5.08 mm
- net Net-(J1005-Pad6): track 0.00 -> 5.08 mm
- net Net-(J1005-Pad4): track 0.00 -> 5.08 mm
- net Net-(J1005-Pad2): track 0.00 -> 5.08 mm
- net Net-(J1003-Pad6): track 0.00 -> 5.08 mm
- net Net-(J1003-Pad4): track 0.00 -> 5.08 mm
- net Net-(J1003-Pad2): track 0.00 -> 5.08 mm
- net Net-(J1007-Pad5): track 0.00 -> 5.08 mm
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- added copper zone on B.Cu, net (none)
Other:
- board size 81.3 x 34.2 mm -> 81.3 x 30.5 mm
- board text added: "07/17"
- board text added: "1"
- board text added: "2"
- board text added: "3"
- board text added: "4"
- board text removed: "FEV 16"
- board text removed: "ICD_BOARD"
