File: ELECTRONICAL_MAIN_BOARD_32/V1-40/ELECTRONICAL_MAIN_BOARD_32_1_42.kicad_pcb (KiCad board)
At the start: 2 copper layers, 88.4 x 99.7 mm, 124 parts, among them J1 SIL1, J2 SIL1, J3 SIL1, J4 SIL1, J5 RJ12, J6 SIL1, J7 SIL1, K1 CONN_3, K2 CONN_3, K3 CONN_3, K4 CONN_3, K5 CONN_3, K6 CONN_3, K7 CONN_3, K8 CONN_2, P1 HE10-16, P10 CONN_2, P11 CONN_2, P14 CAVALIER, P15 CAVALIER, P2 CONN_4, P3 CONN_4, P4 CONN_4, P5 CONN_4, P6 CONN_4, P7 CONN_4, P8 CONN_2, P9 CONN_5, Q1 BSS123, Q2 BSS123, Q3 BSS123, Q4 BSS123, Q5 IRFL9014TRPBF, Q6 2N7002, SW1 SWITCH_X_8, SW2 SW_PUSH_SMALL, SW3 SWITCH_X_8, U1 PIC32MX795F512H, U2 74LVCC3245, U3 74LVCC3245, U4 PCA9306, U5 PCA9306, U6 74LVCC3245, U7 24C512, U8 LM75A, U9 PCF8563, X1 CRYSTAL1

Commit message: MAJ
Routing:
- net /PIC32/PGED1: track 80.7 -> 124.5 mm, vias 2 -> 4
- net /PIC32/PGEC1: track 73.4 -> 116.3 mm, vias 2 -> 4
- net /PIC32/SW1: track 71.4 -> 55.0 mm
- net /PIC32/SW12: track 59.1 -> 72.5 mm
- net Net-(Q6-Pad1): track 1.93 -> 12.1 mm
- net Net-(Q5-Pad1): track 74.7 -> 66.9 mm
- net /PIC32/RST: track 152.3 -> 144.9 mm, vias 6 -> 5
- net /PIC32/SW10: track 44.1 -> 37.9 mm
- net +5V: track 444.9 -> 449.0 mm
- net /5vto3v3/OC2-5V: track 75.2 -> 78.1 mm
- net /PIC32/SW9: track 44.6 -> 41.7 mm
- net GND: track 894.8 -> 892.1 mm
- net /PIC32/SW0: track 56.5 -> 59.0 mm, vias 3 -> 2
- net /PIC32/SW2: track 55.9 -> 58.3 mm
- net /5vto3v3/SDA1: track 47.5 -> 45.6 mm
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Other:
- board text added: "11/2017"
- board text added: "UART-1"
- board text added: "UART-2"
- board text added: "UART-5"
- board text added: "UART-6"

Commit message: MAJ 2018
Parts:
- moved J4 0.28 mm to (120.7, 57.0)
Other:
- board text added: "POWER_MB"
Changed lines of the file:
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@@
-(kicad_pcb (version 4) (host pcbnew 4.0.6)
+(kicad_pcb (version 4) (host pcbnew 4.0.7)
   (general
     (links 329)
@@
     (area 35.496499 53.911499 124.269501 153.987501)
     (thickness 1.6002)
-    (drawings 36)
+    (drawings 37)
     (tracks 2464)
     (zones 0)
@@
     (mod_text_size 1.524 1.524)
     (mod_text_width 0.3048)
-    (pad_size 6 8.5)
-    (pad_drill 4)
+    (pad_size 3.2512 3.2512)
+    (pad_drill 3.2512)
     (pad_to_mask_clearance 0.254)
     (aux_axis_origin 0 0)
     (visible_elements 7FFEF7FF)
     (pcbplotparams
-      (layerselection 0x00030_80000001)
+      (layerselection 0x010f0_80000001)
       (usegerberextensions true)
       (excludeedgelayer true)
@@
     (model TO_SOT_Packages_SMD.3dshapes/SOT-223.wrl
       (at (xyz 0 0 0))
-      (scale (xyz 0.4 0.4 0.4))
-      (rotate (xyz 0 0 0))
+      (scale (xyz 1 1 1))
+      (rotate (xyz 0 0 270))
     )
   )
@@
   )
   (module COLONETTE (layer Dessus)
-    (at 120.61952 57.30748 270)
+    (at 120.7262 57.0484 270)
     (fp_text reference J4 (at 0 0 270) (layer F.SilkS)
       (effects (font (thickness 0.3048)))
@@
       (effects (font (thickness 0.3048)))
     )
-    (pad 1 thru_hole rect (at 0 0 270) (size 7 7) (drill 4.0005 (offset 1 1)) (layers *.Cu)
+    (pad 1 thru_hole rect (at 0 0 270) (size 7.6 7.6) (drill 4.0005 (offset 1 1)) (layers *.Cu)
       (net 92 "Net-(J4-Pad1)"))
     (model f4deb.3dshapes/Colonette1.wrl
@@
     (pad 5 thru_hole circle (at 1.905 0 270) (size 1.7 1.7) (drill 0.8128) (layers *.Cu *.Mask F.SilkS)
       (net 57 /PIC32/PGEC1))
-    (pad 8 thru_hole circle (at 5.08 8.89 270) (size 3.2512 3.2512) (drill 0.8128) (layers *.Cu *.Mask F.SilkS)
+    (pad 8 thru_hole circle (at 5.08 8.89 270) (size 3.2512 3.2512) (drill 3.2512) (layers *.Cu *.Mask F.SilkS)
       (net 94 "Net-(J5-Pad8)"))
-    (pad 7 thru_hole circle (at -5.08 8.89 270) (size 3.2512 3.2512) (drill 0.8128) (layers *.Cu *.Mask F.SilkS)
+    (pad 7 thru_hole circle (at -5.08 8.89 270) (size 3.2512 3.2512) (drill 3.2512) (layers *.Cu *.Mask F.SilkS)
       (net 95 "Net-(J5-Pad7)"))
     (model f4deb.3dshapes/RJ12-COUDE.wrl
@@
     (descr "Connecteur 4 pibs")
     (tags "CONN DEV")
-    (fp_text reference P9 (at 2.63652 4.66598 180) (layer F.SilkS)
+    (fp_text reference P9 (at -5.23748 2.50698 180) (layer F.SilkS)
       (effects (font (size 1.73482 1.08712) (thickness 0.27178)))
     )
@@
       (rotate (xyz 0 0 90))
     )
-    (model Resistors_SMD.3dshapes/R_0603.wrl
-      (at (xyz 0 0 0))
-      (scale (xyz 1 1 1))
-      (rotate (xyz 0 0 0))
-    )
   )
   (module SM0603_Capa (layer Dessus)
@@
     )
   )
+  (gr_text POWER_MB (at 100.584 61.595) (layer F.SilkS)
+    (effects (font (size 2.032 1.524) (thickness 0.3048)))
+  )
   (dimension 88.392 (width 0.3048) (layer Dwgs.User)
