File: POWER_BOARD/V2-30/Power Supply Board.kicad_pcb (KiCad board)
At the start: 2 copper layers, 74.9 x 95.2 mm, 32 parts, among them J1 CONN_02X08, J2 CONN_02X08, J3 CONN_02X08, J4 CONN_02X08, J5 CONN_02X13, K1 CONN_2, K2 CONN_2, K3 CONN_2, K4 CONN_2, K5 COLONETTE, K6 COLONETTE, K7 COLONETTE, K8 COLONETTE, P1 CONN_6, P2 CONN_12, P3 CONN_6, P4 CONN_6, P5 CONN_6, P6 CONN_6, P7 CONN_6, P8 CONN_6, P9 CONN_6

Commit message: MAJ 09/2018
Other:
- board text added: "08/2018"
- board text removed: "02/2018"
Changed lines of the file:
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@@
-(kicad_pcb (version 4) (host pcbnew 4.0.7)
+(kicad_pcb (version 4) (host pcbnew 4.0.5+dfsg1-4)
   (general
     (links 151)
@@
   )
   (layers
-    (0 Composant signal hide)
-    (31 Cuivre signal hide)
+    (0 Composant signal)
+    (31 Cuivre signal)
     (32 B.Adhes user)
     (33 F.Adhes user)
@@
     (visible_elements 7FFEFFFF)
     (pcbplotparams
-      (layerselection 0x01030_80000001)
-      (usegerberextensions false)
+      (layerselection 0x010f0_80000001)
+      (usegerberextensions true)
       (excludeedgelayer true)
       (linewidth 0.150000)
@@
       (psnegative false)
       (psa4output false)
-      (plotreference true)
-      (plotvalue true)
+      (plotreference false)
+      (plotvalue false)
       (plotinvisibletext false)
       (padsonsilk false)
       (subtractmaskfromsilk false)
-      (outputformat 2)
+      (outputformat 1)
       (mirror false)
-      (drillshape 2)
+      (drillshape 0)
       (scaleselection 1)
       (outputdirectory ""))
@@
     (effects (font (size 2.032 1.524) (thickness 0.3048)))
   )
-  (gr_text 02/2018 (at 167.3225 45.9105 270) (layer Composant)
-    (effects (font (size 2.032 1.524) (thickness 0.3048)))
-  )
+  (gr_text 08/2018 (at 167.3225 45.9105 270) (layer Composant)
+    (effects (font (size 2.032 1.524) (thickness 0.3048)))
+  )
