File: POWER_BOARD/V2-30/Power Supply Board.sch (KiCad schematic (older format))
At the start: 32 parts, among them J1 CONN_02X08, J2 CONN_02X08, J3 CONN_02X08, J4 CONN_02X08, J5 CONN_02X13, K1 CONN_2, K2 CONN_2, K3 CONN_2, K4 CONN_2, K5 COLONETTE, K6 COLONETTE, K7 COLONETTE, K8 COLONETTE, P1 CONN_6, P2 CONN_12, P3 CONN_6, P4 CONN_6, P5 CONN_6, P6 CONN_6, P7 CONN_6, P8 CONN_6, P9 CONN_6

Commit message: MAJ 09/2018
Parts:
- D10, D11, D12, D13, D14: symbol LED -> LED-RESCUE-Power_Supply_Board
- R10, R15, R20, R21, R5: symbol R -> R-RESCUE-Power_Supply_Board
Changed lines of the file:
@@
 EESchema Schematic File Version 2
-LIBS:CEN-SCHEMA
+LIBS:Power Supply Board-rescue
 LIBS:power
 LIBS:device
@@
 LIBS:cmos4000
 LIBS:adc-dac
-LIBS:conn
 LIBS:memory
 LIBS:xilinx
@@
 LIBS:contrib
 LIBS:valves
-LIBS:leds
+LIBS:CEN-SCHEMA
 LIBS:Power Supply Board-cache
 EELAYER 25 0
@@
 $EndComp
 $Comp
-L R R15
+L R-RESCUE-Power_Supply_Board R15
 U 1 1 578FC3C1
 P 5775 6650
@@
 $EndComp
 $Comp
-L R R10
+L R-RESCUE-Power_Supply_Board R10
 U 1 1 578FC3C2
 P 5475 6650
@@
 $EndComp
 $Comp
-L R R20
+L R-RESCUE-Power_Supply_Board R20
 U 1 1 578FC3C4
 P 6075 6650
@@
 $EndComp
 $Comp
-L R R21
+L R-RESCUE-Power_Supply_Board R21
 U 1 1 578FC3C5
 P 6375 6650
@@
 $EndComp
 $Comp
-L LED D11
+L LED-RESCUE-Power_Supply_Board D11
 U 1 1 578FC3C6
 P 5475 6350
@@
 $EndComp
 $Comp
-L LED D12
+L LED-RESCUE-Power_Supply_Board D12
 U 1 1 578FC3C7
 P 5775 6350
@@
 $EndComp
 $Comp
-L LED D13
+L LED-RESCUE-Power_Supply_Board D13
 U 1 1 578FC3C9
 P 6075 6350
@@
 $EndComp
 $Comp
-L LED D14
+L LED-RESCUE-Power_Supply_Board D14
 U 1 1 578FC3CA
 P 6375 6350
@@
 $EndComp
 $Comp
-L R R5
+L R-RESCUE-Power_Supply_Board R5
 U 1 1 578FC3D6
 P 5125 6650
@@
 $EndComp
 $Comp
-L LED D10
+L LED-RESCUE-Power_Supply_Board D10
 U 1 1 578FC3D7
 P 5125 6350
