File: POWER_MODULE/V0.40-THN/POWER_MODULE.kicad_pcb (KiCad board)
At the start: 2 copper layers, 84.2 x 30.1 mm, 18 parts, among them P1 CONN_8X2, U1 TRACO-THN-15-1211

Commit message: MAJ 09/2018
Parts:
- removed the P1 at (40.4, 44.3)
- removed the P1 at (69.0, 44.3)
- removed the R3 at (50.6, 41.6)
- removed the R3 at (79.2, 41.6)
- removed the R4 at (48.1, 41.6)
- removed the R4 at (76.6, 41.6)
- removed the R5 at (45.5, 41.6)
- removed the R5 at (74.1, 41.6)
- removed the R6 at (43.0, 41.6)
- removed the R6 at (71.6, 41.6)
- removed the U1 at (59.5, 18.6)
- removed the U1 at (88.1, 18.6)
- added P1: CONN_8X2, f4deb-mod-library:HE10-16-F-2, B.Cu at (84.1, 53.9)
- added P1: CONN_8X2, f4deb-mod-library:HE10-16-F-2, B.Cu at (140.7, 54.0)
- added P1: CONN_8X2, f4deb-mod-library:HE10-16-F-2, B.Cu at (140.7, 85.1)
- added P1: CONN_8X2, f4deb-mod-library:HE10-16-F-2, B.Cu at (112.5, 85.0)
- added P1: CONN_8X2, f4deb-mod-library:HE10-16-F-2, B.Cu at (84.1, 85.0)
- added P1: CONN_8X2, f4deb-mod-library:HE10-16-F-2, B.Cu at (84.1, 116.1)
- added P1: CONN_8X2, f4deb-mod-library:HE10-16-F-2, B.Cu at (112.5, 116.1)
- added P1: CONN_8X2, f4deb-mod-library:HE10-16-F-2, B.Cu at (140.7, 116.1)
- added R3: 0, Resistors_SMD:R_0805, F.Cu at (150.8, 113.5)
- added R3: 0, Resistors_SMD:R_0805, F.Cu at (94.3, 113.4)
- added R3: 0, Resistors_SMD:R_0805, F.Cu at (122.6, 113.4)
- added R3: 0, Resistors_SMD:R_0805, F.Cu at (122.6, 82.4)
- added R3: 0, Resistors_SMD:R_0805, F.Cu at (94.3, 82.4)
- added R3: 0, Resistors_SMD:R_0805, F.Cu at (150.8, 82.4)
- added R3: 0, Resistors_SMD:R_0805, F.Cu at (150.8, 51.3)
- added R3: 0, Resistors_SMD:R_0805, F.Cu at (94.3, 51.2)
- added R4: 0, Resistors_SMD:R_0805, F.Cu at (148.3, 113.5)
- added R4: 0, Resistors_SMD:R_0805, F.Cu at (91.8, 113.4)
- added R4: 0, Resistors_SMD:R_0805, F.Cu at (120.1, 113.4)
- added R4: 0, Resistors_SMD:R_0805, F.Cu at (120.1, 82.4)
- added R4: 0, Resistors_SMD:R_0805, F.Cu at (91.8, 82.4)
- added R4: 0, Resistors_SMD:R_0805, F.Cu at (148.3, 82.4)
- added R4: 0, Resistors_SMD:R_0805, F.Cu at (148.3, 51.3)
- added R4: 0, Resistors_SMD:R_0805, F.Cu at (91.8, 51.2)
- added R5: 0, Resistors_SMD:R_0805, F.Cu at (145.7, 113.5)
- added R5: 0, Resistors_SMD:R_0805, F.Cu at (89.2, 113.4)
- added R5: 0, Resistors_SMD:R_0805, F.Cu at (117.5, 113.4)
- added R5: 0, Resistors_SMD:R_0805, F.Cu at (117.5, 82.4)
- added R5: 0, Resistors_SMD:R_0805, F.Cu at (89.2, 82.4)
- added R5: 0, Resistors_SMD:R_0805, F.Cu at (145.7, 82.4)
- added R5: 0, Resistors_SMD:R_0805, F.Cu at (145.7, 51.3)
- added R5: 0, Resistors_SMD:R_0805, F.Cu at (89.2, 51.2)
- added R6: 0, Resistors_SMD:R_0805, F.Cu at (143.2, 113.5)
- added R6: 0, Resistors_SMD:R_0805, F.Cu at (86.7, 113.4)
- added R6: 0, Resistors_SMD:R_0805, F.Cu at (115.0, 113.4)
- added R6: 0, Resistors_SMD:R_0805, F.Cu at (115.0, 82.4)
- added R6: 0, Resistors_SMD:R_0805, F.Cu at (86.7, 82.4)
- added R6: 0, Resistors_SMD:R_0805, F.Cu at (143.2, 82.4)
- added R6: 0, Resistors_SMD:R_0805, F.Cu at (143.2, 51.3)
- added R6: 0, Resistors_SMD:R_0805, F.Cu at (86.7, 51.2)
- added U1: TRACO-THN-15-1211, f4deb-mod-library:TRACO-THN-15-1211, B.Cu at (103.2, 28.3)
- added U1: TRACO-THN-15-1211, f4deb-mod-library:TRACO-THN-15-1211, B.Cu at (159.7, 28.3)
- added U1: TRACO-THN-15-1211, f4deb-mod-library:TRACO-THN-15-1211, B.Cu at (159.7, 59.4)
- added U1: TRACO-THN-15-1211, f4deb-mod-library:TRACO-THN-15-1211, B.Cu at (131.5, 59.4)
- added U1: TRACO-THN-15-1211, f4deb-mod-library:TRACO-THN-15-1211, B.Cu at (103.2, 59.4)
- added U1: TRACO-THN-15-1211, f4deb-mod-library:TRACO-THN-15-1211, B.Cu at (131.5, 90.4)
- added U1: TRACO-THN-15-1211, f4deb-mod-library:TRACO-THN-15-1211, B.Cu at (159.7, 90.5)
- added U1: TRACO-THN-15-1211, f4deb-mod-library:TRACO-THN-15-1211, B.Cu at (103.2, 90.5)
- U1: footprint f4deb-mod-library:TRACO-THN -> f4deb-mod-library:TRACO-THN-15-1211
- moved R4 100.9 mm to (120.1, 51.2)
- moved R6 100.9 mm to (115.0, 51.2)
- moved P1 100.9 mm to (112.5, 53.9)
- moved R3 100.9 mm to (122.6, 51.2)
- moved R5 100.9 mm to (117.5, 51.2)
- moved U1 100.9 mm to (131.5, 28.3)
Routing:
- net GND: track 289.4 -> 868.1 mm, vias 15 -> 45
- net Net-(R3-Pad2): track 75.9 -> 324.4 mm
- net +BATT: track 55.5 -> 166.4 mm
- net +5VA: track 5.15 -> 15.5 mm
- net +5V: track 5.15 -> 15.5 mm
- net +3V3: track 5.15 -> 15.5 mm
- net +12V: track 5.15 -> 15.5 mm
- net Net-(P1-Pad3): track 3.05 -> 9.14 mm
Other:
- board size 84.2 x 30.1 mm -> 83.7 x 92.1 mm
- board text removed: "V 0-4 POWER_MODULE"
