File: ELECTRONICAL_MAIN_BOARD_32/V1-50/5vto3v3.sch (KiCad schematic (older format))
At the start: 40 parts, among them P14 CAVALIER, P15 CAVALIER, Q1 BSS123, Q2 BSS123, Q3 BSS123, Q4 BSS123, U2 74LVCC3245, U3 74LVCC3245, U4 PCA9306, U5 PCA9306, U6 74LVCC3245, U8 LM75A, U9 PCF8563, X1 CRYSTAL1

Commit message: ICHUB/PCF8574
Parts:
- C12: value C -> 10p
Changed lines of the file:
@@
 P 5150 5900
 F 0 "C12" H 5200 6000 50  0000 L CNN
-F 1 "C" H 5200 5800 50  0000 L CNN
+F 1 "10p" H 5200 5800 50  0000 L CNN
 F 2 "Capacitors_SMD:C_0603" H 5150 5900 60  0001 C CNN
 F 3 "~" H 5150 5900 60  0000 C CNN
