File: PCB_I2C/V0-20/file5D0A7A0F.sch (KiCad schematic (older format))
At the start: 20 parts, among them J501 Conn_01x04, J502 Conn_01x01_Female, J503 Conn_01x01_Female, SW502 SW_Coded_SH-7050, U501 PCF8574A

Commit message: MAJ
Parts:
- R507, R509, R511, R513: value 47k -> 1.5k
Changed lines of the file:
@@
 P 7025 4150
 F 0 "R509" V 6950 4075 50  0000 L CNN
-F 1 "47k" V 7025 4075 50  0000 L CNN
+F 1 "1.5k" V 7025 4075 50  0000 L CNN
 F 2 "Resistor_SMD:R_0805_2012Metric_Pad1.15x1.40mm_HandSolder" V 6955 4150 50  0001 C CNN
 F 3 "~" H 7025 4150 50  0001 C CNN
@@
 P 7175 4150
 F 0 "R511" V 7100 4075 50  0000 L CNN
-F 1 "47k" V 7175 4075 50  0000 L CNN
+F 1 "1.5k" V 7175 4075 50  0000 L CNN
 F 2 "Resistor_SMD:R_0805_2012Metric_Pad1.15x1.40mm_HandSolder" V 7105 4150 50  0001 C CNN
 F 3 "~" H 7175 4150 50  0001 C CNN
@@
 P 6875 4150
 F 0 "R507" V 6800 4075 50  0000 L CNN
-F 1 "47k" V 6875 4075 50  0000 L CNN
+F 1 "1.5k" V 6875 4075 50  0000 L CNN
 F 2 "Resistor_SMD:R_0805_2012Metric_Pad1.15x1.40mm_HandSolder" V 6805 4150 50  0001 C CNN
 F 3 "~" H 6875 4150 50  0001 C CNN
@@
 P 7325 4150
 F 0 "R513" V 7250 4075 50  0000 L CNN
-F 1 "47k" V 7325 4075 50  0000 L CNN
+F 1 "1.5k" V 7325 4075 50  0000 L CNN
 F 2 "Resistor_SMD:R_0805_2012Metric_Pad1.15x1.40mm_HandSolder" V 7255 4150 50  0001 C CNN
 F 3 "~" H 7325 4150 50  0001 C CNN
