File: MOTOR_BOARD_I2C/V0-20-tc9685/MOTOR_BOARD_I2C.kicad_pcb (KiCad board)
At the start: 2 copper layers, 55.1 x 78.7 mm, 120 parts, among them J1 Conn_01x02, J101 Conn_01x03, J102 Conn_01x04, J401 Conn_01x03_Male, J402 Conn_01x03_Male, J403 Conn_01x03_Male, J404 Conn_01x03_Male, J405 Conn_01x03_Male, J406 Conn_01x03_Male, Q201 2N7002, Q202 2N7002, Q203 BTN8982TA, Q204 BTN8982TA, Q401 2N7002, Q402 2N7002, Q403 2N7002, Q404 2N7002, Q405 2N7002, Q406 2N7002, U101 MCP3427-xUN, U102 MCP23017_SS, U103 74HC00, U104 PCA9685PW, U501 74HC02, U502 74HC02

Commit message: RGB_PCA9685
Parts:
- added D101: Vert, LED_SMD:LED_0603_1608Metric_Pad1.05x0.95mm_HandSolder, F.Cu at (184.0, 57.9)
- added D102: Vert, LED_SMD:LED_0603_1608Metric_Pad1.05x0.95mm_HandSolder, F.Cu at (184.0, 60.2)
- added R126: 1k, Resistor_SMD:R_0603_1608Metric_Pad1.05x0.95mm_HandSolder, F.Cu at (180.5, 57.9)
- added R127: 3.3k, Resistor_SMD:R_0603_1608Metric_Pad1.05x0.95mm_HandSolder, F.Cu at (180.5, 60.2)
- Q203, Q204: footprint Package_TO_SOT_SMD:TO-263-7_TabPin4 -> Package_TO_SOT_SMD:TO-263-7_TabPin8
Routing:
- net GND: track 404.6 -> 422.6 mm, vias 25 -> 26
- net +15V: track 103.1 -> 120.7 mm, vias 4 -> 5
- net +5VD: track 308.5 -> 316.8 mm
- net Net-(C207-Pad2): track 31.8 -> 29.5 mm, vias 8 -> 11
- net Net-(C205-Pad2): track 28.2 -> 30.1 mm, vias 8 -> 11
- net Net-(D102-Pad1): track 0.00 -> 1.81 mm
- net Net-(D101-Pad1): track 0.00 -> 1.81 mm
- net /IN1: track 44.4 -> 45.3 mm
- net /IN5: track 65.9 -> 66.5 mm
- added copper zone on B.Cu, net GND
