File: MOTHER_BOARD/V0-10/Main.sch (KiCad schematic (older format))
At the start: 3 parts

Commit message: MAJ mother_board
Parts:
- added J?: USB_OTG, symbol Connector:USB_OTG
- SW? (x3): symbol CEN-SCHEMA:SWITCH_x_4 -> mother_board-rescue:SWITCH_x_4-CEN-SCHEMA
Connections:
- wire segments 39 -> 47
Changed lines of the file:
@@
 encoding utf-8
 Sheet 2 7
-Title ""
-Date ""
-Rev ""
-Comp ""
-Comment1 ""
+Title "MTOHER_BOARD"
+Date "2020-06-21"
+Rev "V0.10"
+Comp "F4DEB-FOCUS ROBOTIQUE"
+Comment1 "Main View"
 Comment2 ""
 Comment3 ""
@@
 $EndDescr
 $Sheet
-S 2100 1275 2675 4700
+S 2100 1275 2125 5425
 U 5EEA4917
 F0 "Main-Pic32MZ" 50
@@
 F13 "SW00" I L 2100 2475 50
 F14 "RST" I L 2100 2725 50
-F15 "PGED1MAIN" I L 2100 3150 50
-F16 "PGEC1MAIN" I L 2100 3225 50
+F15 "PGED1MAIN" I L 2100 2950 50
+F16 "PGEC1MAIN" I L 2100 3025 50
+F17 "LED1MAIN" I R 4225 1375 50
+F18 "LED2MAIN" I R 4225 1475 50
+F19 "RETROLCD" I R 4225 1650 50
+F20 "MainSCL2" I R 4225 2925 50
+F21 "MainSDA2" I R 4225 2850 50
+F22 "MainSDA1" I R 4225 2650 50
+F23 "MainSCL1" I R 4225 2725 50
+F24 "MainSDA3" I R 4225 3050 50
+F25 "MainSCL3" I R 4225 3125 50
+F26 "T1CK" I R 4225 6075 50
+F27 "MainSDA4" I R 4225 3250 50
+F28 "MainSCL4" I R 4225 3325 50
+F29 "MainUART4RX" I R 4225 3950 50
+F30 "MainUART6RX" I R 4225 4450 50
+F31 "MainUART3TX" I R 4225 3725 50
+F32 "MainUART3RX" I R 4225 3650 50
+F33 "MainUART2RX" I R 4225 4150 50
+F34 "MainUART2TX" I R 4225 4225 50
+F35 "MainUART4TX" I R 4225 4025 50
+F36 "MainUART1RX" I R 4225 4625 50
+F37 "MainUART1TX" I R 4225 4700 50
+F38 "MainUART6TX" I R 4225 4525 50
+F39 "MainUART5RX" I R 4225 4825 50
+F40 "MainUART5TX" I R 4225 4900 50
+F41 "SCK2" I L 2100 4625 50
+F42 "SDO2" I L 2100 4700 50
+F43 "SDI2" I L 2100 4775 50
+F44 "SCK5" I L 2100 4925 50
+F45 "SDI5" I L 2100 5075 50
+F46 "DOLCD" I R 4225 1725 50
+F47 "D1LCD" I R 4225 1800 50
+F48 "D2LCD" I R 4225 1875 50
+F49 "D3LCD" I R 4225 1950 50
+F50 "ELCD" I R 4225 2025 50
+F51 "RSLCD" I R 4225 2100 50
+F52 "RWLCD" I R 4225 2175 50
+F53 "IO0" I L 2100 3975 50
+F54 "IO1" I L 2100 4050 50
+F55 "IO2" I L 2100 4125 50
+F56 "IO3" I L 2100 4200 50
+F57 "IO4" I L 2100 4275 50
+F58 "IO5" I L 2100 4350 50
+F59 "IO6" I L 2100 4425 50
+F60 "IO7" I L 2100 4500 50
+F61 "OC4" I L 2100 5525 50
+F62 "OC3" I L 2100 5450 50
+F63 "OC2" I L 2100 5375 50
+F64 "OC1" I L 2100 5300 50
+F65 "OC5" I L 2100 5600 50
+F66 "T2CK" I R 4225 6175 50
+F67 "OC7" I L 2100 5750 50
+F68 "OC6" I L 2100 5675 50
+F69 "AN2" I R 4225 5300 50
+F70 "AN27" I R 4225 5375 50
+F71 "AN28" I R 4225 5450 50
+F72 "AN8" I R 4225 5525 50
+F73 "AN10" I R 4225 5600 50
+F74 "C1RX" I R 4225 5800 50
+F75 "C1TX" I R 4225 5875 50
+F76 "D-" I L 2100 3475 50
+F77 "D+" I L 2100 3375 50
+F78 "USBID" I L 2100 3575 50
+F79 "VBUS" I L 2100 3175 50
+F80 "SDO5" I L 2100 5000 50
 $EndSheet
-$Sheet
-S 7425 2975 1500 2325
-U 5EEA496D
-F0 "Main-buffer" 50
-F1 "Main-Buffer.sch" 50
-$EndSheet
-$Comp
-L CEN-SCHEMA:SWITCH_x_4 SW?
+$Comp
+L mother_board-rescue:SWITCH_x_4-CEN-SCHEMA SW?
 U 1 1 5EEA4C06
 P 1700 2475
@@
 $EndComp
 $Comp
-L CEN-SCHEMA:SWITCH_x_4 SW?
+L mother_board-rescue:SWITCH_x_4-CEN-SCHEMA SW?
 U 1 1 5EEA5452
 P 1700 2075
@@
 $EndComp
 $Comp
-L CEN-SCHEMA:SWITCH_x_4 SW?
+L mother_board-rescue:SWITCH_x_4-CEN-SCHEMA SW?
 U 1 1 5EEA5970
 P 1700 1675
@@
 RST
 Wire Wire Line
-	2100 3150 1850 3150
-Wire Wire Line
-	2100 3225 1850 3225
-Text Label 2050 3150 2    50   ~ 0
+	2100 2950 1575 2950
+Wire Wire Line
+	2100 3025 1575 3025
+Text Label 2050 2950 2    50   ~ 0
 PGED1MAIN
-Text Label 2050 3225 2    50   ~ 0
+Text Label 2050 3025 2    50   ~ 0
 PGEC1MAIN
+$Sheet
+S 7425 2975 1500 2325
+U 5EEA496D
+F0 "Main-buffer" 50
+F1 "Main-Buffer.sch" 50
+$EndSheet
+$Comp
+L Connector:USB_OTG J?
+U 1 1 5F54B541
+P 1075 3375
+F 0 "J?" H 1132 3842 50  0000 C CNN
+F 1 "USB_OTG" H 1132 3751 50  0000 C CNN
+F 2 "" H 1225 3325 50  0001 C CNN
+F 3 " ~" H 1225 3325 50  0001 C CNN
+	1    1075 3375
+	1    0    0    -1
+$EndComp
+Wire Wire Line
+	1375 3175 2100 3175
+Wire Wire Line
+	1375 3375 2100 3375
+Wire Wire Line
+	2100 3475 1375 3475
+Wire Wire Line
+	1375 3575 2100 3575
+Wire Wire Line
+	1075 3775 1075 3825
+Wire Wire Line
+	1075 3825 975  3825
+Wire Wire Line
+	975  3825 975  3775
+Wire Wire Line
+	1075 3825 1075 3875
+Connection ~ 1075 3825
+$Comp
+L power:GND #PWR?
+U 1 1 5F553184
+P 1075 3875
+F 0 "#PWR?" H 1075 3625 50  0001 C CNN
+F 1 "GND" H 1080 3702 50  0000 C CNN
+F 2 "" H 1075 3875 50  0001 C CNN
+F 3 "" H 1075 3875 50  0001 C CNN
+	1    1075 3875
+	1    0    0    -1
+$EndComp
 $EndSCHEMATC

Commit message: Mother Board update
Parts:
- added D?: QLS6B-FKW, LED_SMD:LED_Cree-PLCC6_4.7x1.5mm, symbol LED:QLS6B-FKW
- added D?: AMBER, symbol Device:LED
- added D?: RED, symbol Device:LED
- added J? (x12): Conn_01x03, symbol Connector_Generic:Conn_01x03
- added J?: Conn_01x05, symbol Connector_Generic:Conn_01x05
- added J? (x2): Conn_01x02, symbol Connector_Generic:Conn_01x02
- added J?: Conn_02x08_Odd_Even, symbol Connector_Generic:Conn_02x08_Odd_Even
- added J? (x11): Conn_01x04, symbol Connector_Generic:Conn_01x04
- added J?: RJ12, symbol Connector:RJ12
- added J? (x6): Conn_01x04_Female, symbol Connector:Conn_01x04_Female
- added J? (x6): Conn_01x04_Male, symbol Connector:Conn_01x04_Male
- added R?: 120, symbol Device:R
Connections:
- net labels added: +3.3V, +5VA, +5VD, BD0, BD1, BD2, BD3, BE, BRETRO, BRS, BRW, CONT, IO0, IO1, IO2, IO3, IO4, IO5, IO6, IO7, MainRXMecaTX, MainRXMotorTX, MainSCK, MainSDI, MainSDO, MainTXMechaRX, MainTXMotorRX, PWM4, PWM5, PWM6, PWM7, RESET, RGB1, RGB2, RGB3, SCK5, SCL1, SCL2-5V, SCL3-3V3, SCL4-HS, SDA-HS, SDA1, SDA2-5V, SDA3-3V3, SDA4-HS, SDI5, SDO5, U1RX, U1TX, U2RX, U2TX, U3RX, U3TX, U4RX, U4TX
- net labels removed: PGEC1MAIN, PGED1MAIN, RST
- wire segments 47 -> 307
- no-connect marks 0 -> 1
Other:
- note added: "BUS CAN"
- note added: "CAN\nBUS"
- note added: "COLOR VIEW"
- note added: "Debug\n5V"
- note added: "I2C"
- note added: "I2C-3.3V"
- note added: "I2C-5V"
- note added: "I2C-HighSpeed"
- note added: "I2C\nCOMMON"
- note added: "IO"
- note added: "LCD"
- note added: "Master µC\n3.3v"
- note added: "Master\nPeripheral"
- note added: "Mechanical"
- note added: "Motor"
- note added: "SERVO-MOTOR"
- note added: "SPI\nPeripheral"
- note added: "UART"

Commit message: MOTHER BOARD UPDATE
Parts:
- gave numbers to parts that had none: 47
