File: MOTHER_BOARD/V0-10/motor.sch (KiCad schematic (older format))
At the start: 0 parts

Commit message: Mother Board update
Parts:
- added U?: PIC32MK1024MFC100, symbol F4DEB-LIBRARY-KICAD5:PIC32MK1024MFC100
Connections:
- net labels added: +3V3, GND, IO0, IO1, IO2, IO3, MotorC2RX, MotorC2TX, MotorSCK3, MotorSCL1, MotorSCL2, MotorSCL3, MotorSCL4, MotorSDA1, MotorSDA2, MotorSDA3, MotorSDA4, MotorSDI5, MotorSDO3, MotorSS3, MotorU1RX, MotorU1TX, MotorU2RX, MotorU2TX, MotorU4RX, MotorU4TX, PGEC1, PGED1, PWM1H, PWM1L, PWM2H, PWM2L, PWM3H, PWM3L, PWM4H, PWM4L, PWM5H, PWM5L, PWM6H, PWM6L, QEA1, QEA2, QEA3, QEA4, QEA5, QEA6, QEB1, QEB2, QEB3, QEB4, QEB5, QEB6
- wire segments 0 -> 83
- no-connect marks 0 -> 2

Commit message: MOTHER BOARD UPDATE
Parts:
- removed U?: PIC32MK1024MFC100, symbol F4DEB-LIBRARY-KICAD5:PIC32MK1024MFC100
Connections:
- net labels removed: +3V3, GND, IO0, IO1, IO2, IO3, MotorC2RX, MotorC2TX, MotorSCK3, MotorSCL1, MotorSCL2, MotorSCL3, MotorSCL4, MotorSDA1, MotorSDA2, MotorSDA3, MotorSDA4, MotorSDI5, MotorSDO3, MotorSS3, MotorU1RX, MotorU1TX, MotorU2RX, MotorU2TX, MotorU4RX, MotorU4TX, PGEC1, PGED1, PWM1H, PWM1L, PWM2H, PWM2L, PWM3H, PWM3L, PWM4H, PWM4L, PWM5H, PWM5L, PWM6H, PWM6L, QEA1, QEA2, QEA3, QEA4, QEA5, QEA6, QEB1, QEB2, QEB3, QEB4, QEB5, QEB6
- wire segments 83 -> 0
- no-connect marks 2 -> 0
